File: Edgeberry-Zero.kicad_sch (KiCad schematic)
At the start: 28 parts, among them J1 Molex_KK_1x02_P2.54mm, J2 Raspberry_Pi_2_3, J3 Edgeberry Cartridge Connector, P1 12Vin, Q1 BC547, Q2 BC547, Q3 BC547, SW1 SW_PUSH, U1 24LC256, U2 LM2596S-5.0

Commit message: cleanup
Other:
- note added: "Copyright© 2025 Sanne 'SpuQ' Santens. This design is released under the CERN OHL-W license on GitHub."
- note added: "EDGEBERRY ZERO"
- note added: "Rev. 1.7, early 2025"
- note removed: "Base Board Rev. 1.7, late 2024"
- note removed: "Copyright© 2024 Sanne 'SpuQ' Santens. This design is released under the CERN OHL-W license on GitHub."
- note removed: "EDGEBERRY"
- title: Edgeberry Hardware -> Edgeberry Zero
Changed lines of the file:
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@@
 	(paper "A4")
 	(title_block
-		(title "Edgeberry Hardware")
+		(title "Edgeberry Zero")
 		(date "2024-05-15")
-		(rev "1.5")
+		(rev "1.7")
 	)
 	(junction
@@
 		)
 	)
-	(text "Copyright© 2024 Sanne 'SpuQ' Santens. This design is released under\nthe CERN OHL-W license on GitHub."
+	(text "Copyright© 2025 Sanne 'SpuQ' Santens. This design is released under\nthe CERN OHL-W license on GitHub."
 		(exclude_from_sim no)
 		(at 181.864 178.816 0)
@@
 		)
 	)
-	(text "Base Board Rev. 1.7, late 2024"
+	(text "Rev. 1.7, early 2025"
 		(exclude_from_sim no)
 		(at 181.864 175.006 0)
@@
 		)
 	)
-	(text "EDGEBERRY"
+	(text "EDGEBERRY ZERO"
 		(exclude_from_sim no)
 		(at 181.61 173.736 0)
